Commit message: add test_urdf

File: urdf/kuka.urdf (robot description, URDF)
Before this commit: robot lbr_iiwa, 8 links, 7 joints
Links:
- added link sliding_base, mass 1.0; collision box size=0.4 0.4 0.2; visual box size=0.4 0.4 0.2
Joints:
- added joint base_slider: type prismatic, parent world, child sliding_base, origin xyz=0 0 0 rpy=0 0 0, axis 1 0 0, limit lower=-0.5 upper=0.5 effort=1000 velocity=1.0
- added joint lbr_iiwa_joint_0: type fixed, parent sliding_base, child lbr_iiwa_link_0, origin xyz=0 0 0 rpy=0 0 0
