Commit message: add urdf file of kuka with sliding joint

File: urdf/kuka_with_slide/kuka.urdf (robot description, URDF)
Before this commit: robot lbr_iiwa, 9 links, 9 joints
Links:
- link sliding_base: mass 1.0 -> 0.0; geometry collision box size=6 0.4 0.2; visual box size=6 0.4 0.2
Joints:
- removed joint base_slider
- removed joint lbr_iiwa_joint_0
- added joint sliding_joint: type prismatic, parent sliding_base, child lbr_iiwa_link_0, origin xyz=0 0 0 rpy=0 0 0, axis 1 0 0, limit lower=-0.5 upper=0.5 effort=1000 velocity=1.0

Commit message: fix demo.py and add demo.mp4

File: urdf/kuka_with_slide/kuka.urdf (robot description, URDF)
Before this commit: robot lbr_iiwa, 9 links, 8 joints
Joints:
- joint sliding_joint: limit lower=-0.5 upper=0.5 effort=1000 velocity=1.0 -> lower=-12 upper=12 effort=1000 velocity=1.0
